Commit message: Stop masking RC profiles as Hooke in official launch
The official Autoware branch now treats RC and Hooke as separate vehicle/sensor profiles instead of using Hooke package names for the RC runtime. RC is the current Orin target, so its default launch model, package directories, build lists, and operator docs are named autoracer_rc. Hooke names remain reserved for a future real Hooke profile and the existing Hooke2 adapter assets.

Constraint: RC is the current ARM runtime target and LiDAR remains on the RC C32 sensor-kit path.\nConstraint: Future Hooke support must not reuse RC profile package names or fake empty profile packages.\nRejected: Keep autoracer_hooke_* as the RC profile for compatibility | it preserves the same naming ambiguity that caused operator confusion.\nRejected: Add empty autoracer_hooke_* packages now | no authoritative Hooke sensor/vehicle profile values are migrated yet.\nConfidence: high\nScope-risk: moderate\nDirective: Do not point RC defaults back to autoracer_hooke; add real Hooke profile packages only with real Hooke configuration.\nTested: python3 -m pytest test -q\nTested: git diff --check\nTested: colcon build --symlink-install --packages-select autoracer_rc_description autoracer_rc_launch autoracer_rc_sensor_kit_description autoracer_rc_sensor_kit_launch --cmake-args -DBUILD_TESTING=OFF\nNot-tested: local x86 full Autoware launch smoke; this workstation lacks a complete autoware_launch install, Orin runtime verification follows separately.

File: src/autoracer_rc_description/urdf/vehicle.xacro (robot description, xacro)
@@ -1,5 +1,5 @@
 <?xml version="1.0"?>
 <robot xmlns:xacro="http://ros.org/wiki/xacro">
-  <xacro:property name="vehicle_info" value="${xacro.load_yaml('$(find autoracer_hooke_description)/config/vehicle_info.param.yaml')}"/>
+  <xacro:property name="vehicle_info" value="${xacro.load_yaml('$(find autoracer_rc_description)/config/vehicle_info.param.yaml')}"/>
   <xacro:property name="wheel_base" value="${vehicle_info['/**']['ros__parameters']['wheel_base']}"/>
   <link name="base_link">

File: src/autoracer_rc_sensor_kit_description/urdf/sensor_kit.xacro (robot description, xacro)
@@ -2,5 +2,5 @@
 <robot xmlns:xacro="http://ros.org/wiki/xacro">
   <xacro:macro name="sensor_kit_macro" params="parent x y z roll pitch yaw">
-    <xacro:arg name="config_dir" default="$(find autoracer_hooke_sensor_kit_description)/config"/>
+    <xacro:arg name="config_dir" default="$(find autoracer_rc_sensor_kit_description)/config"/>
     <xacro:property name="sensor_kit_base_link" value="sensor_kit_base_link"/>
     <xacro:property name="calibration" value="${xacro.load_yaml('$(arg config_dir)/sensor_kit_calibration.yaml')}"/>

File: src/autoracer_rc_sensor_kit_description/urdf/sensors.xacro (robot description, xacro)
@@ -1,5 +1,5 @@
 <?xml version="1.0"?>
 <robot xmlns:xacro="http://ros.org/wiki/xacro">
-  <xacro:arg name="config_dir" default="$(find autoracer_hooke_sensor_kit_description)/config"/>
+  <xacro:arg name="config_dir" default="$(find autoracer_rc_sensor_kit_description)/config"/>
   <xacro:property name="calibration" value="${xacro.load_yaml('$(arg config_dir)/sensors_calibration.yaml')}"/>
   <xacro:include filename="sensor_kit.xacro"/>
